File: KiCAD/aks.sch (KiCad schematic (older format))
At the start: 36 parts

Commit message: изменен акселерометр
Parts:
- removed HL3: Светодиод_3Л341Е, MOTOR_VD_VT_HL:Светодиод_SMD_3528, symbol MOTOR:Светодиод
- removed R8: Р1-8В-0.125-20к, MOTOR_RLC:Резистор_SMD_0805_0,125Вт, symbol MOTOR:Резистор_0,125Вт
- added R10, R8: Резистор_0,125Вт, N_RLC:Резистор_SMD_0805_0,125Вт, symbol elements:Резистор_0,125Вт
- added XS11, XS12: VCC, MOTOR_ICO:Отверстие_под_пайку_D1.2, symbol aks-rescue:отверстие_под_пайку-RESCUE-aks
- added XS13: GND, MOTOR_ICO:Отверстие_под_пайку_D1.2, symbol aks-rescue:отверстие_под_пайку-RESCUE-aks
- C3, C4, C5, C6, C7: footprint MOTOR_RLC:Конденсатор_SMD_1812 -> N_RLC:Конденсатор_SMD_0805
- DD1: footprint MOTOR_DD:Микросхема_5559ИНхх -> N_DD:SO-8_RS485_CAN_Milandr_OTK
- HL1, HL2: footprint MOTOR_VD_VT_HL:Светодиод_SMD_3528 -> N_VD_HL:Светодиод_SMD_0603
- VD1: footprint MOTOR_VD_VT_HL:Диод_2Д663А95(КТ-99-1) -> N_VD_HL:Диод_BAR43CFILM_SOT-23
- XS8: value VCC -> res
Connections:
- net labels added: EN1, Ep, GND_in, PB2, PD7
- net labels removed: GND1, Ucc
- no-connect marks 33 -> 28
Other:
- moved on the sheet: XS1, XS10, XS2, XS3, XS4, XS5, XS9
